File: KiCad/VoltReadDevice/VoltReadDevice.kicad_sch (KiCad schematic)
At the start: 6 parts, among them J1 Conn_PinHeader_1x04_P2.54mm_H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, J2 Conn_PinHeader_1x04_P2.54mm_H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, J3 Conn_PinHeader_1x02_P2.54mm_H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, U1 ATtiny412-SS

Commit message: v2.4 - Finished KiCad Design
Parts:
- added J4: Conn_PinHeader_1x02_P2.54mm_Horizontal_SMD, fab:PinHeader_UPDI_01x02_P2.54mm_Horizontal_SMD, symbol Fab Library:Conn_PinHeader_1x02_P2.54mm_Horizontal_SMD
Connections:
- net at J3.1: now also J4.2
- net at J3.2: now also J4.1
Other:
- moved on the sheet: J3
Changed lines of the file:
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@@
+    (stroke (width 0) (type default) (color 0 0 0 0))
+  )
+  (wire (pts (xy 173.99 81.915) (xy 175.895 81.915))
     (stroke (width 0) (type default) (color 0 0 0 0))
   )
@@
   )
   (wire (pts (xy 131.445 112.395) (xy 144.78 112.395))
+    (stroke (width 0) (type default) (color 0 0 0 0))
+  )
+  (wire (pts (xy 173.99 79.375) (xy 175.895 79.375))
     (stroke (width 0) (type default) (color 0 0 0 0))
   )
@@
     (pin "4")
   )
-  (symbol (lib_id "Fab Library:Conn_PinHeader_1x02_P2.54mm_Horizontal_SMD") (at 170.815 81.915 180) (unit 1)
+  (symbol (lib_id "Fab Library:Conn_PinHeader_1x02_P2.54mm_Horizontal_SMD") (at 180.975 81.915 180) (unit 1)
     (in_bom yes) (on_board yes) (fields_autoplaced)
-    (property "Reference" "J3" (id 0) (at 171.45 80.6449 0)
+    (property "Reference" "J3" (id 0) (at 181.61 80.6449 0)
       (effects (font (size 1.27 1.27)) (justify right))
     )
-    (property "Value" "Conn_PinHeader_1x02_P2.54mm_Horizontal_SMD" (id 1) (at 171.45 81.9149 0)
+    (property "Value" "Conn_PinHeader_1x02_P2.54mm_Horizontal_SMD" (id 1) (at 181.61 81.9149 0)
       (effects (font (size 1.27 1.27)) (justify right) hide)
     )
-    (property "Footprint" "fab:PinHeader_UPDI_01x02_P2.54mm_Horizontal_SMD" (id 2) (at 170.815 81.915 0)
+    (property "Footprint" "fab:PinHeader_UPDI_01x02_P2.54mm_Horizontal_SMD" (id 2) (at 180.975 81.915 0)
       (effects (font (size 1.27 1.27)) hide)
     )
-    (property "Datasheet" "~" (id 3) (at 170.815 81.915 0)
+    (property "Datasheet" "~" (id 3) (at 180.975 81.915 0)
       (effects (font (size 1.27 1.27)) hide)
     )
@@
     )
     (property "Datasheet" "https://optoelectronics.liteon.com/upload/download/DS-22-98-0002/LTST-C150CKT.pdf" (id 3) (at 160.655 99.06 0)
+      (effects (font (size 1.27 1.27)) hide)
+    )
+    (pin "1")
+    (pin "2")
+  )
+  (symbol (lib_id "Fab Library:Conn_PinHeader_1x02_P2.54mm_Horizontal_SMD") (at 168.91 79.375 0) (unit 1)
+    (in_bom yes) (on_board yes) (fields_autoplaced)
+    (property "Reference" "J4" (id 0) (at 169.9768 76.2 0))
+    (property "Value" "Conn_PinHeader_1x02_P2.54mm_Horizontal_SMD" (id 1) (at 168.275 79.3751 0)
+      (effects (font (size 1.27 1.27)) (justify right) hide)
+    )
+    (property "Footprint" "fab:PinHeader_UPDI_01x02_P2.54mm_Horizontal_SMD" (id 2) (at 168.91 79.375 0)
+      (effects (font (size 1.27 1.27)) hide)
+    )
+    (property "Datasheet" "~" (id 3) (at 168.91 79.375 0)
       (effects (font (size 1.27 1.27)) hide)
     )
@@
       (reference "J3") (unit 1) (value "Conn_PinHeader_1x02_P2.54mm_Horizontal_SMD") (footprint "fab:PinHeader_UPDI_01x02_P2.54mm_Horizontal_SMD")
     )
+    (path "/7e78ef60-e353-441f-9dfb-ec02cef9b164"
+      (reference "J4") (unit 1) (value "Conn_PinHeader_1x02_P2.54mm_Horizontal_SMD") (footprint "fab:PinHeader_UPDI_01x02_P2.54mm_Horizontal_SMD")
+    )
     (path "/c5318030-0c39-492d-82c8-f5e8f484d6df"
